File: SynchroDriverD/SynchroDriverD.kicad_pcb (KiCad board)
At the start: 2 copper layers, 100 x 100 mm, 201 parts, among them J1 SYNC, J2 POWER, J3 ROLL, J4 PITCH, J5 YAW, J6 NEEDLES, J7 FLAG, Q1 SIS990, Q2 SIS990, Q3 SIS990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

Commit message: PCB layout
Parts:
- moved R70 0.30 mm to (159.0, 129.7)
- moved R52 0.28 mm to (132.9, 108.9)
- moved R63 0.27 mm to (132.9, 124.7)
- moved R64 0.27 mm to (132.9, 132.6)
- moved R50 0.25 mm to (132.9, 93.2)
- moved R62 0.25 mm to (132.9, 116.8)
- moved R51 0.23 mm to (132.9, 101.0)
- moved R10 0.22 mm to (132.9, 85.2)
- moved R9 0.22 mm to (132.9, 77.2)
- moved R48 0.22 mm to (132.9, 110.6)
- moved R8 0.20 mm to (132.9, 69.5)
- moved C65 0.20 mm to (156.7, 129.7)
- moved C68 0.20 mm to (157.8, 126.4)
- moved R6 0.14 mm to (132.9, 86.9)
- moved R7 0.14 mm to (132.9, 78.9)
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Routing:
- net /NeedleDriver1/VREF: track 0.00 -> 95.6 mm, vias 0 -> 6
- net Net-(D2-A): track 0.00 -> 33.8 mm, vias 0 -> 2
- net +36V: track 0.00 -> 30.2 mm
- net Net-(C28-Pad2): track 0.00 -> 23.5 mm
- net Net-(C27-Pad2): track 0.00 -> 22.1 mm
- net Net-(Q1A-S): track 0.00 -> 21.3 mm, vias 0 -> 2
- net Net-(Q7A-S): track 0.00 -> 20.8 mm, vias 0 -> 2
- net Net-(Q4A-S): track 0.00 -> 20.6 mm, vias 0 -> 2
- net Net-(Q6A-S): track 0.00 -> 20.4 mm, vias 0 -> 2
- net Net-(C36-Pad2): track 0.00 -> 19.9 mm
- net Net-(Q9A-S): track 0.00 -> 19.2 mm, vias 0 -> 2
- net Net-(Q3A-S): track 0.00 -> 19.0 mm, vias 0 -> 2
- net Net-(U9-GLC): track 0.00 -> 17.4 mm
- net GND: track 0.00 -> 17.2 mm, vias 0 -> 9
- net Net-(Q2A-S): track 0.00 -> 16.9 mm, vias 0 -> 2
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- added copper zone on F.Cu, net /SingleSynchroDriver1/PHASE_A_OUT
- added copper zone on F.Cu, net /SingleSynchroDriver1/PHASE_B_OUT
- added copper zone on F.Cu, net /SingleSynchroDriver1/PHASE_C_OUT
- added copper zone on F.Cu, net /SingleSynchroDriver2/PHASE_A_OUT
- added copper zone on F.Cu, net /SingleSynchroDriver2/PHASE_B_OUT
- added copper zone on F.Cu, net /SingleSynchroDriver2/PHASE_C_OUT
- added copper zone on F.Cu, net /SingleSynchroDriver3/PHASE_A_OUT
- added copper zone on F.Cu, net /SingleSynchroDriver3/PHASE_B_OUT
- added copper zone on F.Cu, net /SingleSynchroDriver3/PHASE_C_OUT
- added copper zone on F.Cu, net Net-(Q1A-S)
- added copper zone on F.Cu, net Net-(Q2A-S)
- added copper zone on F.Cu, net Net-(Q3A-S)
- added copper zone on F.Cu, net Net-(Q4A-S)
- added copper zone on F.Cu, net Net-(Q5A-S)
- added copper zone on F.Cu, net Net-(Q6A-S)
- added copper zone on F.Cu, net Net-(Q7A-S)
- added copper zone on F.Cu, net Net-(Q8A-S)
- added copper zone on F.Cu, net Net-(Q9A-S)
