File: SynchroDriverD/Pots.kicad_sch (KiCad schematic)
At the start: 9 parts

Commit message: Mouser parts, layout changes
Parts:
- RV1, RV2, RV3, RV4, RV5, RV6, RV7, RV8, RV9: Mouser (none) -> 652-PTV09A4030FB103
Changed lines of the file:
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@@
+			)
+		)
+		(property "Mouser" "652-PTV09A4030FB103"
+			(at 121.92 144.78 0)
+			(effects
+				(font
+					(size 1.27 1.27)
+				)
+				(hide yes)
 			)
 		)
@@
 			)
 		)
+		(property "Mouser" "652-PTV09A4030FB103"
+			(at 121.92 128.27 0)
+			(effects
+				(font
+					(size 1.27 1.27)
+				)
+				(hide yes)
+			)
+		)
 		(pin "MP"
 		)
@@
 			)
 		)
+		(property "Mouser" "652-PTV09A4030FB103"
+			(at 121.92 62.23 0)
+			(effects
+				(font
+					(size 1.27 1.27)
+				)
+				(hide yes)
+			)
+		)
 		(pin "MP"
 		)
@@
 			)
 		)
+		(property "Mouser" "652-PTV09A4030FB103"
+			(at 121.92 78.74 0)
+			(effects
+				(font
+					(size 1.27 1.27)
+				)
+				(hide yes)
+			)
+		)
 		(pin "MP"
 		)
@@
 		)
 		(property "MPN" "PTV09A4030FB103"
+			(at 121.92 95.25 0)
+			(effects
+				(font
+					(size 1.27 1.27)
+				)
+				(hide yes)
+			)
+		)
+		(property "Mouser" "652-PTV09A4030FB103"
 			(at 121.92 95.25 0)
 			(effects
@@
 			)
 		)
+		(property "Mouser" "652-PTV09A4030FB103"
+			(at 121.92 161.29 0)
+			(effects
+				(font
+					(size 1.27 1.27)
+				)
+				(hide yes)
+			)
+		)
 		(pin "MP"
 		)
@@
 			)
 		)
+		(property "Mouser" "652-PTV09A4030FB103"
+			(at 121.92 29.21 0)
+			(effects
+				(font
+					(size 1.27 1.27)
+				)
+				(hide yes)
+			)
+		)
 		(pin "MP"
 		)
@@
 			)
 		)
+		(property "Mouser" "652-PTV09A4030FB103"
+			(at 121.92 111.76 0)
+			(effects
+				(font
+					(size 1.27 1.27)
+				)
+				(hide yes)
+			)
+		)
 		(pin "MP"
 		)
@@
 			(at 121.92 45.72 0)
 			(effects
+				(font
+					(size 1.27 1.27)
+				)
+				(hide yes)
+			)
+		)
+		(property "Mouser" "652-PTV09A4030FB103"
+			(at 121.92 45.72 0)
+			(effects
