File: SynchroDriverD/FlagDriver.kicad_sch (KiCad schematic)
At the start: 0 parts

Commit message: Ad flag drive circuit
Parts:
- added Q10: MMBTA42, Package_TO_SOT_SMD:SOT-23, symbol Transistor_BJT:MMBTA42
- added Q11: MMBTA92, Package_TO_SOT_SMD:SOT-23, symbol Transistor_BJT:MMBTA92
- added R3, R76: 10K, Resistor_SMD:R_0603_1608Metric, symbol Device:R_Small_US
- added R4: 22K, Resistor_SMD:R_0603_1608Metric, symbol Device:R_Small_US
- added R77: 2.2K, Resistor_SMD:R_0603_1608Metric, symbol Device:R_Small_US
Connections:
- new net: Q10.1 (B), R76.1
- new net: Q10.3 (C), R4.1
- new net: Q11.3 (C), R77.2
- new net: Q11.1 (B), R3.1, R4.2
- new net +36V: Q11.2 (E), R3.2
- new net GND: Q10.2 (E)
- new net IN: R76.2
- new net OUT: R77.1
Other:
- note added: "2mA"

Commit message: Tweaks after first build
Parts:
- Q10: Mouser (none) -> 637-MMBTA42
- Q11: Mouser (none) -> 637-MMBTA92
Changed lines of the file:
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@@
+			)
+		)
+		(property "Mouser" "637-MMBTA42"
+			(at 104.14 95.25 0)
+			(effects
+				(font
+					(size 1.27 1.27)
+				)
+				(hide yes)
 			)
 		)
@@
 			(at 106.68 72.39 0)
 			(effects
+				(font
+					(size 1.27 1.27)
+				)
+				(hide yes)
+			)
+		)
+		(property "Mouser" "637-MMBTA92"
+			(at 106.68 72.39 0)
+			(effects
