File: SynchroDriverD/NeedleDriver.kicad_sch (KiCad schematic)
At the start: 15 parts, among them U5 LM324

Commit message: Tweaks after first build
Parts:
- R23, R24: value 10K -> 20K
- U5: Mouser (none) -> 863-LM324DR2G
Other:
- note added: "1.1V"
- note removed: "(1.65V)"
Changed lines of the file:
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@@
 		)
 	)
-	(text "(1.65V)"
+	(text "1.1V"
 		(exclude_from_sim no)
 		(at 102.108 85.09 0)
@@
 			)
 		)
-		(property "Value" "10K"
+		(property "Value" "20K"
 			(at 121.666 57.15 90)
 			(effects
@@
 			)
 		)
-		(property "Value" "10K"
+		(property "Value" "20K"
 			(at 121.666 109.22 90)
 			(effects
@@
 		)
 		(property "Description" "Low-Power, Quad-Operational Amplifiers, DIP-14/SOIC-14/SSOP-14"
+			(at 119.38 125.73 0)
+			(effects
+				(font
+					(size 1.27 1.27)
+				)
+				(hide yes)
+			)
+		)
+		(property "Mouser" "863-LM324DR2G"
 			(at 119.38 125.73 0)
 			(effects
@@
 			(at 119.38 73.66 0)
 			(effects
+				(font
+					(size 1.27 1.27)
+				)
+				(hide yes)
+			)
+		)
+		(property "Mouser" "863-LM324DR2G"
+			(at 119.38 73.66 0)
+			(effects

Commit message: Firmware PWM frequency fix. Synchro bodge. Needle value changes
Parts:
- C25, C26: value DNI -> 0.1uF
- R17, R18: value 10K -> DNI
- R19, R20: value 0 -> 1K
Other:
- note removed: "Optional RC"
Changed lines of the file:
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@@
 	(generator_version "9.0")
 	(paper "A4")
-	(text "Optional RC"
-		(exclude_from_sim no)
-		(at 70.612 67.056 0)
-		(effects
-			(font
-				(size 1.27 1.27)
-			)
-		)
-	)
 	(text "1.1V"
 		(exclude_from_sim no)
 		(at 102.108 85.09 0)
-		(effects
-			(font
-				(size 1.27 1.27)
-			)
-		)
-	)
-	(text "Optional RC"
-		(exclude_from_sim no)
-		(at 70.612 119.126 0)
 		(effects
 			(font
@@
 			)
 		)
-		(property "Value" "DNI"
+		(property "Value" "0.1uF"
 			(at 79.502 76.962 0)
 			(effects
@@
 			)
 		)
-		(property "Value" "10K"
+		(property "Value" "DNI"
 			(at 67.31 83.312 0)
 			(effects
@@
 			)
 		)
-		(property "Value" "0"
+		(property "Value" "1K"
 			(at 73.406 121.92 90)
 			(effects
@@
 			)
 		)
-		(property "Value" "0"
+		(property "Value" "1K"
 			(at 73.406 69.85 90)
 			(effects
@@
 			)
 		)
-		(property "Value" "DNI"
+		(property "Value" "0.1uF"
 			(at 79.502 129.032 0)
 			(effects
@@
 			)
 		)
-		(property "Value" "10K"
+		(property "Value" "DNI"
 			(at 67.31 133.35 0)
 			(effects
