File: SynchroDriverD/SingleSynchroDriver.kicad_sch (KiCad schematic)
At the start: 36 parts, among them Q1 SIS990, Q2 SIS990, Q3 SIS990, U3 74LV14, U8 DRV8300

Commit message: Swap DRV8300 for DRV8300DI, change ref in
Parts:
- removed U3: 74LV14, Active:SOP127P620X175-14, symbol 74xx:74LV14
- added R78, R81, R84: 0, Passive:RESC1608X55, symbol Device:R_Small_US
- U8: value DRV8300 -> DRV8300DI
Connections:
- net INA: now also R78.1
- net INB: now also R81.1
- net INC: now also R84.1
- net at U8.4 (INLA): now also R78.2
- net at U8.5 (INLB): now also R81.2
- net at U8.6 (INLC): now also R84.2

Commit message: Tweaks after first build
Parts:
- C13, C14, C15, C19, C20, C21: Mouser (none) -> 187-CL31A106KBHNNNE
- C16, C17, C18: value DNI -> 560pF
- L1, L2, L3: Mouser (none) -> 871-B82472G4224M
- Q1, Q2, Q3: Mouser (none) -> 78-SIS990DN-T1-GE3
- R11, R12, R13: value DNI -> 5.6
- U8: Mouser (none) -> 595-DRV8300DIPWR
Changed lines of the file:
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@@
 			)
 		)
-		(property "Value" "DNI"
+		(property "Value" "560pF"
 			(at 212.852 102.362 0)
 			(effects
@@
 			)
 		)
+		(property "Mouser" "871-B82472G4224M"
+			(at 214.63 107.95 0)
+			(effects
+				(font
+					(size 1.27 1.27)
+				)
+				(hide yes)
+			)
+		)
 		(pin "1"
 		)
@@
 			)
 		)
-		(property "Value" "DNI"
+		(property "Value" "560pF"
 			(at 213.614 118.364 0)
 			(effects
@@
 			)
 		)
-		(property "Value" "DNI"
+		(property "Value" "5.6"
 			(at 210.82 112.522 0)
 			(effects
@@
 			)
 		)
+		(property "Mouser" "78-SIS990DN-T1-GE3"
+			(at 151.13 129.54 0)
+			(effects
+				(font
+					(size 1.27 1.27)
+				)
+				(hide yes)
+			)
+		)
 		(pin "1"
 		)
@@
 			)
 		)
+		(property "Mouser" "187-CL31A106KBHNNNE"
+			(at 219.71 129.54 0)
+			(effects
+				(font
+					(size 1.27 1.27)
+				)
+				(hide yes)
+			)
+		)
 		(pin "2"
 		)
@@
 			)
 		)
+		(property "Mouser" "187-CL31A106KBHNNNE"
+			(at 219.71 99.06 0)
+			(effects
+				(font
+					(size 1.27 1.27)
+				)
+				(hide yes)
+			)
+		)
 		(pin "2"
 		)
@@
 			)
 		)
+		(property "Mouser" "871-B82472G4224M"
+			(at 214.63 123.19 0)
+			(effects
+				(font
+					(size 1.27 1.27)
+				)
+				(hide yes)
+			)
+		)
 		(pin "1"
 		)
@@
 					(size 1.27 1.27)
 				)
+				(hide yes)
+			)
+		)
+		(property "Mouser" "871-B82472G4224M"
+			(at 214.63 92.71 0)
+			(effects
+				(font
+					(size 1.27 1.27)
+				)
+				(hide yes)
 			)
 		)
@@
 			)
 		)
+		(property "Mouser" "187-CL31A106KBHNNNE"
+			(at 177.8 71.12 0)
+			(effects
+				(font
+					(size 1.27 1.27)
+				)
+				(hide yes)
+			)
+		)
 		(pin "2"
 		)
@@
 			)
 		)
-		(property "Value" "DNI"
+		(property "Value" "5.6"
 			(at 210.82 127.762 0)
 			(effects
@@
 			)
 		)
-		(property "Value" "DNI"
+		(property "Value" "560pF"
 			(at 213.614 133.604 0)
 			(effects
@@
 			)
 		)
+		(property "Mouser" "187-CL31A106KBHNNNE"
+			(at 219.71 114.3 0)
+			(effects
+				(font
+					(size 1.27 1.27)
+				)
+				(hide yes)
+			)
+		)
 		(pin "2"
 		)
@@
 			)
 		)
-		(property "Value" "DNI"
+		(property "Value" "5.6"
 			(at 210.82 97.282 0)
 			(effects
@@
 			)
 		)
+		(property "Mouser" "78-SIS990DN-T1-GE3"
+			(at 189.23 129.54 0)
+			(effects
+				(font
+					(size 1.27 1.27)
+				)
+				(hide yes)
+			)
+		)
 		(pin "1"
 		)
@@
 			)
 		)
+		(property "Mouser" "78-SIS990DN-T1-GE3"
+			(at 170.18 129.54 0)
+			(effects
+				(font
+					(size 1.27 1.27)
+				)
+				(hide yes)
+			)
+		)
 		(pin "1"
 		)
@@
 			)
 		)
+		(property "Mouser" "78-SIS990DN-T1-GE3"
+			(at 170.18 101.6 0)
+			(effects
+				(font
+					(size 1.27 1.27)
+				)
+				(hide yes)
+			)
+		)
 		(pin "1"
 		)
@@
 			)
 		)
+		(property "Mouser" "78-SIS990DN-T1-GE3"
+			(at 189.23 116.84 0)
+			(effects
+				(font
+					(size 1.27 1.27)
+				)
+				(hide yes)
+			)
+		)
 		(pin "1"
 		)
@@
 			)
 		)
+		(property "Mouser" "187-CL31A106KBHNNNE"
+			(at 158.75 71.12 0)
+			(effects
+				(font
+					(size 1.27 1.27)
+				)
+				(hide yes)
+			)
+		)
 		(pin "2"
 		)
@@
 			)
 		)
+		(property "Mouser" "78-SIS990DN-T1-GE3"
+			(at 151.13 86.36 0)
+			(effects
+				(font
+					(size 1.27 1.27)
+				)
+				(hide yes)
+			)
+		)
 		(pin "1"
 		)
@@
 			)
 		)
+		(property "Mouser" "187-CL31A106KBHNNNE"
+			(at 196.85 71.12 0)
+			(effects
+				(font
+					(size 1.27 1.27)
+				)
+				(hide yes)
+			)
+		)
 		(pin "2"
 		)
@@
 			(effects
 				(font
+					(size 1.27 1.27)
+				)
+				(hide yes)
+			)
+		)
+		(property "Mouser" "595-DRV8300DIPWR"
+			(at 106.68 78.74 0)
+			(effects
+				(font

Commit message: Firmware PWM frequency fix. Synchro bodge. Needle value changes
Parts:
- added R91, R94, R97: 10K, Passive:RESC1608X55, symbol Device:R_Small_US
Connections:
- net GND: now also R91.1, R94.1, R97.1
- net INA: now also R97.2
- net INB: now also R94.2
- net INC: now also R91.2
Other:
- note added: "BODGE"
