File: SynchroDriverAS/SynchroDriverAS.kicad_pcb (KiCad board)
At the start: 2 copper layers, 46 x 30 mm, 42 parts, among them J1 POWER, J2 INPUTS, J3 OUTPUTS, U1 L165, U2 L165, U3 L165

Commit message: Layout for analog 3-phase pcb
Parts:
- moved C11 4.74 mm to (112.5, 89.2), turned to 180 degrees
- moved C15 4.56 mm to (123.6, 89.2), turned to 180 degrees
- moved C7 3.86 mm to (102.2, 89.2), turned to 180 degrees
- moved J1 1.80 mm to (134.7, 85.0)
- moved R5 1.00 mm to (106.5, 89.2)
- moved R11 0.60 mm to (128.3, 89.2)
Routing:
- net +15V: track 0.00 -> 43.9 mm, vias 0 -> 3
- net -15V: track 0.00 -> 43.7 mm, vias 0 -> 3
- net /PhaseDriver1/VREF: track 0.00 -> 39.7 mm
- net /PhaseDriver3/IN: track 0.00 -> 33.8 mm, vias 0 -> 1
- net /PhaseDriver2/IN: track 0.00 -> 21.9 mm, vias 0 -> 1
- net /PhaseDriver1/IN: track 0.00 -> 9.89 mm, vias 0 -> 1
- net GND: track 0.00 -> 6.90 mm, vias 0 -> 11
- net Net-(U2--): track 0.00 -> 4.96 mm
- net Net-(U1--): track 0.00 -> 4.95 mm
- net Net-(U3--): track 0.00 -> 4.87 mm
- net VDD: track 0.00 -> 4.44 mm
- net Net-(C15-Pad1): track 0.00 -> 2.20 mm
- net Net-(C7-Pad1): track 0.00 -> 1.80 mm
- net Net-(C11-Pad1): track 0.00 -> 1.80 mm
- added copper zone on B.Cu, net +15V
- added copper zone on B.Cu, net -15V
- added copper zone on F.Cu, net /PhaseDriver1/OUT
- added copper zone on F.Cu, net /PhaseDriver2/OUT
- added copper zone on F.Cu, net /PhaseDriver3/OUT
- added copper zone on B.Cu, net GND
- added copper zone on F.Cu, net GND
Other:
- board text added: "+V"
- board text added: "-V"
- board text added: "3-PHASE PWM TO ANALOG"
- board text added: "GND"
- board text added: "IN VCC"
- board text added: "IN1"
- board text added: "IN2"
- board text added: "IN3"
- board text added: "INPUT"
- board text added: "OUT1"
- board text added: "OUT2"
- board text added: "OUT3"
- board text added: "POWER"
- board text added: "©2025 TUBE TIME"
