File: SynchroDriverDS/SynchroDriverDS.kicad_sch (KiCad schematic)
At the start: 5 parts, among them J1 POWER, J2 CTRL, J3 Conn_01x04

Commit message: Update digital single synchro pcb
Parts:
- added H1, H2, H3, H4: MountingHole_Pad, MountingHole:MountingHole_3.2mm_M3_DIN965_Pad, symbol Mechanical:MountingHole_Pad
Connections:
- net GND: now also H1.1, H2.1, H3.1, H4.1
