File: SynchroDriverDS/SingleSynchroDriver.kicad_sch (KiCad schematic)
At the start: 41 parts, among them Q1 2N7002, Q2 2N7002, Q3 2N7002, Q4 SIS990, Q5 SIS990, Q6 SIS990, U1 DRV8300

Commit message: Swap DRV8300 for DRV8300DI, change ref in
Parts:
- removed Q1, Q2, Q3: 2N7002, Package_TO_SOT_SMD:SOT-23, symbol Transistor_FET:2N7002
- R1, R2, R3: value 4.7K -> 0
- U1: value DRV8300 -> DRV8300DI
Connections:
- net +12V: no longer R1.2, R2.2, R3.2
- net INA: now also R1.2
- net INB: now also R2.2
- net INC: now also R3.2
Other:
- moved on the sheet: R1, R2, R3

Commit message: Tweaks after first build
Parts:
- C10, C11, C12: value DNI -> 560pF
- R10, R11, R12: value DNI -> 5.6
Changed lines of the file:
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@@
 			)
 		)
-		(property "Value" "DNI"
+		(property "Value" "560pF"
 			(at 212.852 102.362 0)
 			(effects
@@
 			)
 		)
-		(property "Value" "DNI"
+		(property "Value" "560pF"
 			(at 213.614 118.364 0)
 			(effects
@@
 			)
 		)
-		(property "Value" "DNI"
+		(property "Value" "5.6"
 			(at 210.82 112.522 0)
 			(effects
@@
 			)
 		)
-		(property "Value" "DNI"
+		(property "Value" "5.6"
 			(at 210.82 127.762 0)
 			(effects
@@
 			)
 		)
-		(property "Value" "DNI"
+		(property "Value" "560pF"
 			(at 213.614 133.604 0)
 			(effects
@@
 			)
 		)
-		(property "Value" "DNI"
+		(property "Value" "5.6"
 			(at 210.82 97.282 0)
 			(effects
